Commit message: some changes

File: examples/objects/bottle.urdf (robot description, URDF)
Before this commit: robot urdf_robot, 1 links, 0 joints
Links:
- link base_link: geometry collision cylinder length=0.04 radius=0.03; visual mesh filename=bottle/bottle.obj scale=0.009 0.009 0.009

File: examples/objects/chips_can.urdf (robot description, URDF)
Before this commit: robot urdf_robot, 1 links, 0 joints
Links:
- link base_link: geometry collision mesh filename=chips_can/chips_can.obj scale=0.6 0.6 0.6; visual mesh filename=chips_can/chips_can.obj

File: examples/objects/cube.urdf (robot description, URDF)
Before this commit: robot cube.urdf, 1 links, 0 joints
Links:
- link baseLink: geometry collision box size=.10 .05 .15; visual mesh filename=cube/cube.obj scale=.10 .05 .15

Commit message: some fixes to get good grasping

File: examples/objects/bottle.urdf (robot description, URDF)
Before this commit: robot urdf_robot, 1 links, 0 joints
Links:
- link base_link: geometry collision mesh filename=bottle/bottle.obj scale=0.0085 0.0085 0.0085; visual mesh filename=bottle/bottle.obj scale=0.009 0.009 0.009

File: examples/objects/chips_can.urdf (robot description, URDF)
Before this commit: robot urdf_robot, 1 links, 0 joints
Links:
- link base_link: geometry collision mesh filename=chips_can/chips_can.obj scale=0.9 0.9 0.9; visual mesh filename=chips_can/chips_can.obj
