Commit message: Added Single Visualization and Save Image interface

File: examples/objects/chef_can.urdf (robot description, URDF)
Before this commit: robot urdf_robot, 1 links, 0 joints
Links:
- link base_link: geometry collision mesh filename=chef_can/chef_can.obj scale=0.9 0.9 0.9; visual mesh filename=chef_can/chef_can.obj

File: examples/objects/cylinder.urdf (robot description, URDF)
Before this commit: robot urdf_robot, 1 links, 0 joints
Links:
- link base_link: mass 1 -> .1; geometry collision cylinder length=0.3 radius=0.3; visual cylinder length=0.3 radius=0.3

File: examples/objects/mug.urdf (robot description, URDF)
Before this commit: robot urdf_robot, 1 links, 0 joints
Links:
- link base_link: geometry collision mesh filename=mug/mug.obj scale=0.9 0.9 0.9; visual mesh filename=mug/mug.obj

File: examples/objects/plate.urdf (robot description, URDF)
Before this commit: robot urdf_robot, 1 links, 0 joints
Links:
- link base_link: mass 1 -> .1; geometry collision mesh filename=plate/plate.obj scale=0.9 0.9 0.9; visual mesh filename=plate/plate.obj

File: examples/objects/tomato_soup_can.urdf (robot description, URDF)
Before this commit: robot urdf_robot, 1 links, 0 joints
Links:
- link base_link: mass 1 -> .1; geometry collision mesh filename=tomato_soup_can/tomato_soup_can.obj scale=0.9 0.9 0.9; visual mesh filename=tomato_soup_can/tomato_soup_can.obj

Commit message: added image saving

File: examples/objects/chef_can.urdf (robot description, URDF)
Before this commit: robot urdf_robot, 1 links, 0 joints
Links:
- link base_link: mass .1 -> .2

File: examples/objects/mug.urdf (robot description, URDF)
Before this commit: robot urdf_robot, 1 links, 0 joints
Links:
- link base_link: geometry collision mesh filename=mug/mug.obj scale=0.8 0.8 0.8; visual mesh filename=mug/mug.obj
